File: VIOBOARD/VIOBOARD.sch (KiCad schematic (older format))
At the start: 5 parts, among them J1 Screw_Terminal_1x04, J2 Conn_02x02_Top_Bottom, J8 TEST_1P, J9 TEST_1P, SW1 BOARD_RESET

Commit message: Libraries modified as part of the BBB cape developement.
Parts:
- J8, J9: symbol conn:TEST_1P -> VIOBOARD-rescue:TEST_1P-conn
- SW1: symbol switches:SW_SPST -> VIOBOARD-rescue:SW_SPST-switches
Changed lines of the file:
@@
 	3850 3300 4150 3300
 $Comp
-L switches:SW_SPST SW1
+L VIOBOARD-rescue:SW_SPST-switches SW1
 U 1 1 596BEDF5
 P 8250 4300
@@
 $EndComp
 $Comp
-L conn:TEST_1P J8
+L VIOBOARD-rescue:TEST_1P-conn J8
 U 1 1 596A4B02
 P 2000 3700
@@
 $EndComp
 $Comp
-L conn:TEST_1P J9
+L VIOBOARD-rescue:TEST_1P-conn J9
 U 1 1 596A5164
 P 4150 3300
