File: VIOBOARD/5V_POWER_SUPPLY.sch (KiCad schematic (older format))
At the start: 15 parts, among them J11 TEST_1P, U9 PTN78000WAH

Commit message: Libraries modified as part of the BBB cape developement.
Parts:
- C44, C45, C46, C48, C50, C51: symbol device:C_Small -> VIOBOARD-rescue:C_Small-device
- C47, C49: symbol device:CP1_Small -> VIOBOARD-rescue:CP1_Small-device
- J11: symbol conn:TEST_1P -> VIOBOARD-rescue:TEST_1P-conn
- R66, R67, R68, R69: symbol device:R -> VIOBOARD-rescue:R-device
Changed lines of the file:
@@
 	5950 3550 5800 3550
 $Comp
-L device:CP1_Small C47
+L VIOBOARD-rescue:CP1_Small-device C47
 U 1 1 59600D6D
 P 5350 4300
@@
 $EndComp
 $Comp
-L device:CP1_Small C49
+L VIOBOARD-rescue:CP1_Small-device C49
 U 1 1 59600DB8
 P 8450 3650
@@
 $EndComp
 $Comp
-L device:C_Small C46
+L VIOBOARD-rescue:C_Small-device C46
 U 1 1 5960118D
 P 5000 4300
@@
 $EndComp
 $Comp
-L device:C_Small C48
+L VIOBOARD-rescue:C_Small-device C48
 U 1 1 596013BE
 P 8100 3650
@@
 $EndComp
 $Comp
-L device:C_Small C45
+L VIOBOARD-rescue:C_Small-device C45
 U 1 1 596018F1
 P 4650 4300
@@
 $EndComp
 $Comp
-L device:C_Small C50
+L VIOBOARD-rescue:C_Small-device C50
 U 1 1 5960193C
 P 7350 3650
@@
 Connection ~ 8100 3550
 $Comp
-L device:C_Small C44
+L VIOBOARD-rescue:C_Small-device C44
 U 1 1 5966B067
 P 4250 4300
@@
 $EndComp
 $Comp
-L device:C_Small C51
+L VIOBOARD-rescue:C_Small-device C51
 U 1 1 5966B0FE
 P 7700 3650
@@
 Connection ~ 8900 3550
 $Comp
-L conn:TEST_1P J11
+L VIOBOARD-rescue:TEST_1P-conn J11
 U 1 1 596A4484
 P 8900 3550
@@
 	5000 4400 5000 4500
 $Comp
-L device:R R66
+L VIOBOARD-rescue:R-device R66
 U 1 1 5A41F8D0
 P 4250 3850
@@
 $EndComp
 $Comp
-L device:R R67
+L VIOBOARD-rescue:R-device R67
 U 1 1 5A41F95A
 P 4650 3850
@@
 $EndComp
 $Comp
-L device:R R68
+L VIOBOARD-rescue:R-device R68
 U 1 1 5A41F9B4
 P 5000 3850
@@
 $EndComp
 $Comp
-L device:R R69
+L VIOBOARD-rescue:R-device R69
 U 1 1 5A41FA09
 P 5350 3850

Commit message: Schematics cleanup.  Gerbers for the latest manufacturing release.
Parts:
- R45: value 21K 1% -> 21K; symbol CUSTOM_COMPONENTS:R_C -> VIOBOARD-rescue:R_C-CUSTOM_COMPONENTS
- R66, R67, R68, R69: value 0 1% -> 0
- U9: symbol CUSTOM_COMPONENTS:PTN78000WAH -> VIOBOARD-rescue:PTN78000WAH-CUSTOM_COMPONENTS
Changed lines of the file:
@@
 $EndDescr
 $Comp
-L CUSTOM_COMPONENTS:PTN78000WAH U9
+L VIOBOARD-rescue:PTN78000WAH-CUSTOM_COMPONENTS U9
 U 1 1 59600C27
 P 6100 3850
@@
 	7700 4500 7700 3750
 $Comp
-L CUSTOM_COMPONENTS:R_C R45
+L VIOBOARD-rescue:R_C-CUSTOM_COMPONENTS R45
 U 1 1 59602B03
 P 6800 4250
 F 0 "R45" V 6800 4250 50  0000 C CNN
-F 1 "21K 1%" V 6700 4250 39  0000 C CNN
+F 1 "21K" V 6700 4250 39  0000 C CNN
 F 2 "Resistors_SMD:R_0805" V 6730 4250 50  0001 C CNN
 F 3 "" H 6800 4250 50  0001 C CNN
@@
 P 4250 3850
 F 0 "R66" V 4250 3850 50  0000 C CNN
-F 1 "0 1%" V 4150 3850 39  0000 C CNN
+F 1 "0" V 4150 3850 39  0000 C CNN
 F 2 "Resistors_SMD:R_0805" V 4180 3850 50  0001 C CNN
 F 3 "" H 4250 3850 50  0001 C CNN
@@
 P 4650 3850
 F 0 "R67" V 4650 3850 50  0000 C CNN
-F 1 "0 1%" V 4550 3850 39  0000 C CNN
+F 1 "0" V 4550 3850 39  0000 C CNN
 F 2 "Resistors_SMD:R_0805" V 4580 3850 50  0001 C CNN
 F 3 "" H 4650 3850 50  0001 C CNN
@@
 P 5000 3850
 F 0 "R68" V 5000 3850 50  0000 C CNN
-F 1 "0 1%" V 4900 3850 39  0000 C CNN
+F 1 "0" V 4900 3850 39  0000 C CNN
 F 2 "Resistors_SMD:R_0805" V 4930 3850 50  0001 C CNN
 F 3 "" H 5000 3850 50  0001 C CNN
@@
 P 5350 3850
 F 0 "R69" V 5350 3850 50  0000 C CNN
-F 1 "0 1%" V 5250 3850 39  0000 C CNN
+F 1 "0" V 5250 3850 39  0000 C CNN
 F 2 "Resistors_SMD:R_0805" V 5280 3850 50  0001 C CNN
 F 3 "" H 5350 3850 50  0001 C CNN
