File: VIOBOARD/AI_INPUT.sch (KiCad schematic (older format))
At the start: 37 parts, among them U5 MCP6004_C

Commit message: Libraries modified as part of the BBB cape developement.
Parts:
- C21, C22, C23, C24, C52, C53, C54, C55, C56, C57, C58, C59: symbol device:C_Small -> VIOBOARD-rescue:C_Small-device
- R78, R79, R80, R81, R82, R83, R84, R85: symbol device:R_Small -> VIOBOARD-rescue:R_Small-device
Changed lines of the file:
@@
 $EndComp
 $Comp
-L device:C_Small C22
+L VIOBOARD-rescue:C_Small-device C22
 U 1 1 5961A41D
 P 6100 5900
@@
 $EndComp
 $Comp
-L device:C_Small C23
+L VIOBOARD-rescue:C_Small-device C23
 U 1 1 5961A498
 P 6600 6100
@@
 $EndComp
 $Comp
-L device:C_Small C24
+L VIOBOARD-rescue:C_Small-device C24
 U 1 1 5961A67E
 P 7000 6350
@@
 $EndComp
 $Comp
-L device:C_Small C21
+L VIOBOARD-rescue:C_Small-device C21
 U 1 1 59659490
 P 6450 5700
@@
 $EndComp
 $Comp
-L device:C_Small C56
+L VIOBOARD-rescue:C_Small-device C56
 U 1 1 5A42EDCC
 P 2250 1400
@@
 $EndComp
 $Comp
-L device:C_Small C54
+L VIOBOARD-rescue:C_Small-device C54
 U 1 1 5A42EF31
 P 2150 1200
@@
 $EndComp
 $Comp
-L device:C_Small C52
+L VIOBOARD-rescue:C_Small-device C52
 U 1 1 5A42EF9B
 P 2050 1000
@@
 $EndComp
 $Comp
-L device:C_Small C58
+L VIOBOARD-rescue:C_Small-device C58
 U 1 1 5A42F0E8
 P 2350 1600
@@
 $EndComp
 $Comp
-L device:C_Small C53
+L VIOBOARD-rescue:C_Small-device C53
 U 1 1 5A4302AC
 P 1700 3700
@@
 $EndComp
 $Comp
-L device:C_Small C55
+L VIOBOARD-rescue:C_Small-device C55
 U 1 1 5A430379
 P 1800 3900
@@
 $EndComp
 $Comp
-L device:C_Small C57
+L VIOBOARD-rescue:C_Small-device C57
 U 1 1 5A4303E3
 P 1900 4100
@@
 $EndComp
 $Comp
-L device:C_Small C59
+L VIOBOARD-rescue:C_Small-device C59
 U 1 1 5A430450
 P 2000 4300
@@
 $EndComp
 $Comp
-L device:R_Small R80
+L VIOBOARD-rescue:R_Small-device R80
 U 1 1 5A4441CC
 P 2600 2100
@@
 $EndComp
 $Comp
-L device:R_Small R82
+L VIOBOARD-rescue:R_Small-device R82
 U 1 1 5A4446E8
 P 2800 2250
@@
 $EndComp
 $Comp
-L device:R_Small R78
+L VIOBOARD-rescue:R_Small-device R78
 U 1 1 5A444761
 P 2250 3500
@@
 $EndComp
 $Comp
-L device:R_Small R79
+L VIOBOARD-rescue:R_Small-device R79
 U 1 1 5A44574A
 P 2450 3350
@@
 $EndComp
 $Comp
-L device:R_Small R81
+L VIOBOARD-rescue:R_Small-device R81
 U 1 1 5A44607D
 P 2650 3200
@@
 $EndComp
 $Comp
-L device:R_Small R83
+L VIOBOARD-rescue:R_Small-device R83
 U 1 1 5A4465C4
 P 2850 3050
@@
 Connection ~ 2000 3050
 $Comp
-L device:R_Small R84
+L VIOBOARD-rescue:R_Small-device R84
 U 1 1 5A44A740
 P 3000 2400
@@
 $EndComp
 $Comp
-L device:R_Small R85
+L VIOBOARD-rescue:R_Small-device R85
 U 1 1 5A44A7CE
 P 3200 2550

Commit message: Schematics cleanup.  Gerbers for the latest manufacturing release.
Parts:
- R20, R22, R24, R28: value 910 1% -> 910; symbol CUSTOM_COMPONENTS:R_C -> VIOBOARD-rescue:R_C-CUSTOM_COMPONENTS
- R21, R23, R26, R30: value 8.2K 1% -> 8K2; symbol CUSTOM_COMPONENTS:R_C -> VIOBOARD-rescue:R_C-CUSTOM_COMPONENTS
- R25, R27, R29, R31, R32, R33, R34, R35: symbol CUSTOM_COMPONENTS:R_C -> VIOBOARD-rescue:R_C-CUSTOM_COMPONENTS
- R78, R79, R80, R81, R82, R83, R84, R85: value 1K 1% -> 1K
- U5: symbol CUSTOM_COMPONENTS:MCP6004_C -> VIOBOARD-rescue:MCP6004_C-CUSTOM_COMPONENTS; DKPN MCP6004T-I/SLCT-ND -> 296-43775-1-ND; MFGPN MCP6004T-I/SL -> TLV4333IDR
Changed lines of the file:
@@
 AI_IN_ICD_4
 $Comp
-L CUSTOM_COMPONENTS:R_C R31
+L VIOBOARD-rescue:R_C-CUSTOM_COMPONENTS R31
 U 1 1 59279937
 P 4900 1050
@@
 $EndComp
 $Comp
-L CUSTOM_COMPONENTS:R_C R29
+L VIOBOARD-rescue:R_C-CUSTOM_COMPONENTS R29
 U 1 1 592799BE
 P 4700 1300
@@
 $EndComp
 $Comp
-L CUSTOM_COMPONENTS:R_C R27
+L VIOBOARD-rescue:R_C-CUSTOM_COMPONENTS R27
 U 1 1 592799E1
 P 4500 1550
@@
 $EndComp
 $Comp
-L CUSTOM_COMPONENTS:R_C R25
+L VIOBOARD-rescue:R_C-CUSTOM_COMPONENTS R25
 U 1 1 592799FE
 P 4300 1800
@@
 $EndComp
 $Comp
-L CUSTOM_COMPONENTS:R_C R35
+L VIOBOARD-rescue:R_C-CUSTOM_COMPONENTS R35
 U 1 1 5927DE6A
 P 8700 1900
@@
 $EndComp
 $Comp
-L CUSTOM_COMPONENTS:R_C R34
+L VIOBOARD-rescue:R_C-CUSTOM_COMPONENTS R34
 U 1 1 5927DEBD
 P 8400 1900
@@
 $EndComp
 $Comp
-L CUSTOM_COMPONENTS:R_C R33
+L VIOBOARD-rescue:R_C-CUSTOM_COMPONENTS R33
 U 1 1 5927DF1A
 P 8100 1900
@@
 $EndComp
 $Comp
-L CUSTOM_COMPONENTS:R_C R32
+L VIOBOARD-rescue:R_C-CUSTOM_COMPONENTS R32
 U 1 1 5927DF65
 P 7800 1900
@@
 $EndComp
 $Comp
-L CUSTOM_COMPONENTS:R_C R28
+L VIOBOARD-rescue:R_C-CUSTOM_COMPONENTS R28
 U 1 1 59269CC3
 P 4600 3500
 F 0 "R28" V 4600 3450 39  0000 L CNN
-F 1 "910 1%" V 4700 3400 39  0000 L CNN
+F 1 "910" V 4700 3400 39  0000 L CNN
 F 2 "Resistors_SMD:R_0805" H 4600 3500 50  0001 C CNN
 F 3 "" H 4600 3500 50  0001 C CNN
@@
 $EndComp
 $Comp
-L CUSTOM_COMPONENTS:R_C R24
+L VIOBOARD-rescue:R_C-CUSTOM_COMPONENTS R24
 U 1 1 5926A016
 P 4200 3500
 F 0 "R24" V 4200 3450 39  0000 L CNN
-F 1 "910 1%" V 4300 3400 39  0000 L CNN
+F 1 "910" V 4300 3400 39  0000 L CNN
 F 2 "Resistors_SMD:R_0805" H 4200 3500 50  0001 C CNN
 F 3 "" H 4200 3500 50  0001 C CNN
@@
 $EndComp
 $Comp
-L CUSTOM_COMPONENTS:R_C R22
+L VIOBOARD-rescue:R_C-CUSTOM_COMPONENTS R22
 U 1 1 5926A0B7
 P 3800 3500
 F 0 "R22" V 3800 3450 39  0000 L CNN
-F 1 "910 1%" V 3900 3400 39  0000 L CNN
+F 1 "910" V 3900 3400 39  0000 L CNN
 F 2 "Resistors_SMD:R_0805" H 3800 3500 50  0001 C CNN
 F 3 "" H 3800 3500 50  0001 C CNN
@@
 $EndComp
 $Comp
-L CUSTOM_COMPONENTS:R_C R20
+L VIOBOARD-rescue:R_C-CUSTOM_COMPONENTS R20
 U 1 1 5926A29C
 P 3400 3500
 F 0 "R20" V 3400 3450 39  0000 L CNN
-F 1 "910 1%" V 3500 3400 39  0000 L CNN
+F 1 "910" V 3500 3400 39  0000 L CNN
 F 2 "Resistors_SMD:R_0805" H 3400 3500 50  0001 C CNN
 F 3 "" H 3400 3500 50  0001 C CNN
@@
 $EndComp
 $Comp
-L CUSTOM_COMPONENTS:R_C R30
+L VIOBOARD-rescue:R_C-CUSTOM_COMPONENTS R30
 U 1 1 5926B5E4
 P 4750 3750
 F 0 "R30" V 4750 3700 39  0000 L CNN
-F 1 "8.2K 1%" V 4850 3650 39  0000 L CNN
+F 1 "8K2" V 4850 3650 39  0000 L CNN
 F 2 "Resistors_SMD:R_0805" H 4750 3750 50  0001 C CNN
 F 3 "" H 4750 3750 50  0001 C CNN
@@
 $EndComp
 $Comp
-L CUSTOM_COMPONENTS:R_C R26
+L VIOBOARD-rescue:R_C-CUSTOM_COMPONENTS R26
 U 1 1 5926B6A5
 P 4350 3750
 F 0 "R26" V 4350 3700 39  0000 L CNN
-F 1 "8.2K 1%" V 4450 3650 39  0000 L CNN
+F 1 "8K2" V 4450 3650 39  0000 L CNN
 F 2 "Resistors_SMD:R_0805" H 4350 3750 50  0001 C CNN
 F 3 "" H 4350 3750 50  0001 C CNN
@@
 $EndComp
 $Comp
-L CUSTOM_COMPONENTS:R_C R23
+L VIOBOARD-rescue:R_C-CUSTOM_COMPONENTS R23
 U 1 1 5926B849
 P 3950 3750
 F 0 "R23" V 3950 3700 39  0000 L CNN
-F 1 "8.2K 1%" V 4050 3650 39  0000 L CNN
+F 1 "8K2" V 4050 3650 39  0000 L CNN
 F 2 "Resistors_SMD:R_0805" H 3950 3750 50  0001 C CNN
 F 3 "" H 3950 3750 50  0001 C CNN
@@
 $EndComp
 $Comp
-L CUSTOM_COMPONENTS:R_C R21
+L VIOBOARD-rescue:R_C-CUSTOM_COMPONENTS R21
 U 1 1 5926B90E
 P 3550 3750
 F 0 "R21" V 3550 3700 39  0000 L CNN
-F 1 "8.2K 1%" V 3650 3650 39  0000 L CNN
+F 1 "8K2" V 3650 3650 39  0000 L CNN
 F 2 "Resistors_SMD:R_0805" H 3550 3750 50  0001 C CNN
 F 3 "" H 3550 3750 50  0001 C CNN
@@
 Vinc-
 $Comp
-L CUSTOM_COMPONENTS:MCP6004_C U5
+L VIOBOARD-rescue:MCP6004_C-CUSTOM_COMPONENTS U5
 U 1 1 5926460F
 P 6000 4700
@@
 F 2 "Housings_SOIC:SOIC-14_3.9x8.7mm_Pitch1.27mm" H 6000 4700 60  0001 C CNN
 F 3 "" H 6000 4700 60  0001 C CNN
-F 4 "MCP6004T-I/SLCT-ND" H 6000 4700 60  0001 C CNN "DKPN"
-F 5 "MCP6004T-I/SL" H 6000 4700 60  0001 C CNN "MFGPN"
+F 4 "296-43775-1-ND" H 6000 4700 60  0001 C CNN "DKPN"
+F 5 "TLV4333IDR" H 6000 4700 60  0001 C CNN "MFGPN"
 	1    6000 4700
 	1    0    0    -1
@@
 P 2600 2100
 F 0 "R80" V 2600 2050 39  0000 L CNN
-F 1 "1K 1%" V 2500 2050 39  0000 L CNN
+F 1 "1K" V 2500 2050 39  0000 L CNN
 F 2 "Resistors_SMD:R_0805" H 2600 2100 50  0001 C CNN
 F 3 "" H 2600 2100 50  0001 C CNN
@@
 P 2800 2250
 F 0 "R82" V 2800 2200 39  0000 L CNN
-F 1 "1K 1%" V 2700 2200 39  0000 L CNN
+F 1 "1K" V 2700 2200 39  0000 L CNN
 F 2 "Resistors_SMD:R_0805" H 2800 2250 50  0001 C CNN
 F 3 "" H 2800 2250 50  0001 C CNN
@@
 P 2250 3500
 F 0 "R78" V 2250 3450 39  0000 L CNN
-F 1 "1K 1%" V 2150 3450 39  0000 L CNN
+F 1 "1K" V 2150 3450 39  0000 L CNN
 F 2 "Resistors_SMD:R_0805" H 2250 3500 50  0001 C CNN
 F 3 "" H 2250 3500 50  0001 C CNN
@@
 P 2450 3350
 F 0 "R79" V 2450 3300 39  0000 L CNN
-F 1 "1K 1%" V 2350 3300 39  0000 L CNN
+F 1 "1K" V 2350 3300 39  0000 L CNN
 F 2 "Resistors_SMD:R_0805" H 2450 3350 50  0001 C CNN
 F 3 "" H 2450 3350 50  0001 C CNN
@@
 P 2650 3200
 F 0 "R81" V 2650 3150 39  0000 L CNN
-F 1 "1K 1%" V 2550 3150 39  0000 L CNN
+F 1 "1K" V 2550 3150 39  0000 L CNN
 F 2 "Resistors_SMD:R_0805" H 2650 3200 50  0001 C CNN
 F 3 "" H 2650 3200 50  0001 C CNN
@@
 P 2850 3050
 F 0 "R83" V 2850 3000 39  0000 L CNN
-F 1 "1K 1%" V 2750 3000 39  0000 L CNN
+F 1 "1K" V 2750 3000 39  0000 L CNN
 F 2 "Resistors_SMD:R_0805" H 2850 3050 50  0001 C CNN
 F 3 "" H 2850 3050 50  0001 C CNN
@@
 P 3000 2400
 F 0 "R84" V 3000 2350 39  0000 L CNN
-F 1 "1K 1%" V 2900 2350 39  0000 L CNN
+F 1 "1K" V 2900 2350 39  0000 L CNN
 F 2 "Resistors_SMD:R_0805" H 3000 2400 50  0001 C CNN
 F 3 "" H 3000 2400 50  0001 C CNN
@@
 P 3200 2550
 F 0 "R85" V 3200 2500 39  0000 L CNN
-F 1 "1K 1%" V 3100 2500 39  0000 L CNN
+F 1 "1K" V 3100 2500 39  0000 L CNN
 F 2 "Resistors_SMD:R_0805" H 3200 2550 50  0001 C CNN
 F 3 "" H 3200 2550 50  0001 C CNN
