File: VIOBOARD/COMM_PWR_DEC.sch (KiCad schematic (older format))
At the start: 4 parts

Commit message: Libraries modified as part of the BBB cape developement.
Parts:
- C10, C11, C12, C13: symbol device:C_Small -> VIOBOARD-rescue:C_Small-device
Changed lines of the file:
@@
 	4550 1500 4550 1550
 $Comp
-L device:C_Small C10
+L VIOBOARD-rescue:C_Small-device C10
 U 1 1 595E9A0A
 P 4850 1350
@@
 $EndComp
 $Comp
-L device:C_Small C11
+L VIOBOARD-rescue:C_Small-device C11
 U 1 1 595E9A57
 P 5100 1350
@@
 $EndComp
 $Comp
-L device:C_Small C12
+L VIOBOARD-rescue:C_Small-device C12
 U 1 1 595E9A72
 P 5350 1350
@@
 $EndComp
 $Comp
-L device:C_Small C13
+L VIOBOARD-rescue:C_Small-device C13
 U 1 1 595E9A9B
 P 5600 1350

Commit message: Schematics cleanup.  Gerbers for the latest manufacturing release.
Changed lines of the file:
@@
 $Descr A4 11693 8268
 encoding utf-8
-Sheet 5 21
+Sheet 4 21
 Title "Vic's IO BOARD V1.0"
 Date "2018-09-03"
@@
 $EndComp
 Wire Wire Line
-	4550 1200 6200 1200
+	4550 1200 4850 1200
 Wire Wire Line
 	4550 1500 4550 1550
@@
 Connection ~ 5600 1500
 Wire Wire Line
-	6200 1500 4550 1500
+	6200 1500 5600 1500
 Text HLabel 6200 1500 2    35   Output ~ 0
 VSS_COMM
+Wire Wire Line
+	4850 1200 5100 1200
+Wire Wire Line
+	5100 1200 5350 1200
+Wire Wire Line
+	5350 1200 5600 1200
+Wire Wire Line
+	5600 1200 6200 1200
+Wire Wire Line
+	4850 1500 4550 1500
+Wire Wire Line
+	5100 1500 4850 1500
+Wire Wire Line
+	5350 1500 5100 1500
+Wire Wire Line
+	5600 1500 5350 1500
 $EndSCHEMATC
