File: VIOBOARD/DIGITAL_OUT.sch (KiCad schematic (older format))
At the start: 23 parts, among them J7 Screw_Terminal_1x04

Commit message: Libraries modified as part of the BBB cape developement.
Parts:
- D20, D21, D22, D23: symbol device:D_ALT -> VIOBOARD-rescue:D_ALT-device
- LED6, LED7, LED8, LED9: symbol device:LED_ALT -> VIOBOARD-rescue:LED_ALT-device
- R61, R62, R63, R64: symbol device:R -> VIOBOARD-rescue:R-device
- R86, R87, R88, R89: symbol device:R_Small -> VIOBOARD-rescue:R_Small-device
Changed lines of the file:
@@
 D_OUT4
 $Comp
-L device:LED_ALT LED6
+L VIOBOARD-rescue:LED_ALT-device LED6
 U 1 1 59302CA1
 P 5600 4700
@@
 Connection ~ 5600 4550
 $Comp
-L device:LED_ALT LED7
+L VIOBOARD-rescue:LED_ALT-device LED7
 U 1 1 59302F1A
 P 5950 4900
@@
 $EndComp
 $Comp
-L device:LED_ALT LED8
+L VIOBOARD-rescue:LED_ALT-device LED8
 U 1 1 59302F59
 P 6300 5100
@@
 $EndComp
 $Comp
-L device:LED_ALT LED9
+L VIOBOARD-rescue:LED_ALT-device LED9
 U 1 1 59302FEE
 P 6650 5300
@@
 Connection ~ 1100 2950
 $Comp
-L device:D_ALT D20
+L VIOBOARD-rescue:D_ALT-device D20
 U 1 1 599AAE85
 P 8250 4550
@@
 $EndComp
 $Comp
-L device:D_ALT D21
+L VIOBOARD-rescue:D_ALT-device D21
 U 1 1 599AB498
 P 8000 4750
@@
 $EndComp
 $Comp
-L device:D_ALT D22
+L VIOBOARD-rescue:D_ALT-device D22
 U 1 1 599AB524
 P 7750 4950
@@
 $EndComp
 $Comp
-L device:D_ALT D23
+L VIOBOARD-rescue:D_ALT-device D23
 U 1 1 599AB59A
 P 7500 5150
@@
 DOUT4
 $Comp
-L device:R R61
+L VIOBOARD-rescue:R-device R61
 U 1 1 5A41B942
 P 8650 4550
@@
 $EndComp
 $Comp
-L device:R R62
+L VIOBOARD-rescue:R-device R62
 U 1 1 5A41B9C8
 P 8650 4750
@@
 $EndComp
 $Comp
-L device:R R63
+L VIOBOARD-rescue:R-device R63
 U 1 1 5A41BA36
 P 8650 4950
@@
 $EndComp
 $Comp
-L device:R R64
+L VIOBOARD-rescue:R-device R64
 U 1 1 5A41BA9B
 P 8650 5150
@@
 	5600 4550 8100 4550
 $Comp
-L device:R_Small R86
+L VIOBOARD-rescue:R_Small-device R86
 U 1 1 5A44DD62
 P 6350 5800
@@
 $EndComp
 $Comp
-L device:R_Small R87
+L VIOBOARD-rescue:R_Small-device R87
 U 1 1 5A44DEF4
 P 6450 6000
@@
 $EndComp
 $Comp
-L device:R_Small R88
+L VIOBOARD-rescue:R_Small-device R88
 U 1 1 5A44DF67
 P 6550 6200
@@
 $EndComp
 $Comp
-L device:R_Small R89
+L VIOBOARD-rescue:R_Small-device R89
 U 1 1 5A44DFDD
 P 6650 6400

Commit message: Schematics cleanup.  Gerbers for the latest manufacturing release.
Parts:
- R49, R50, R51, R52: value 470 1% -> 470; symbol CUSTOM_COMPONENTS:R_C -> VIOBOARD-rescue:R_C-CUSTOM_COMPONENTS
- R61, R62, R63, R64: value 100 1% -> 100
- R86, R87, R88, R89: value 4.7K 1% -> 4K7
- TLPA1, TLPB1: symbol CUSTOM_COMPONENTS:TLP222A-2-C -> VIOBOARD-rescue:TLP222A-2-C-CUSTOM_COMPONENTS
Changed lines of the file:
@@
 Connection ~ 6650 5150
 $Comp
-L CUSTOM_COMPONENTS:TLP222A-2-C TLPA1
+L VIOBOARD-rescue:TLP222A-2-C-CUSTOM_COMPONENTS TLPA1
 U 1 1 5968740A
 P 4100 4850
@@
 $EndComp
 $Comp
-L CUSTOM_COMPONENTS:TLP222A-2-C TLPB1
+L VIOBOARD-rescue:TLP222A-2-C-CUSTOM_COMPONENTS TLPB1
 U 1 1 59687553
 P 5600 3800
@@
 	6300 2800 6300 4950
 $Comp
-L CUSTOM_COMPONENTS:R_C R49
+L VIOBOARD-rescue:R_C-CUSTOM_COMPONENTS R49
 U 1 1 59986459
 P 1800 2650
 F 0 "R49" V 1800 2650 39  0000 C CNN
-F 1 "470 1%" V 1750 2400 39  0000 C CNN
+F 1 "470" V 1750 2400 39  0000 C CNN
 F 2 "Resistors_SMD:R_0805" V 1730 2650 50  0001 C CNN
 F 3 "" H 1800 2650 50  0001 C CNN
@@
 $EndComp
 $Comp
-L CUSTOM_COMPONENTS:R_C R50
+L VIOBOARD-rescue:R_C-CUSTOM_COMPONENTS R50
 U 1 1 59986558
 P 1800 2750
 F 0 "R50" V 1800 2750 39  0000 C CNN
-F 1 "470 1%" V 1750 2500 39  0000 C CNN
+F 1 "470" V 1750 2500 39  0000 C CNN
 F 2 "Resistors_SMD:R_0805" V 1730 2750 50  0001 C CNN
 F 3 "" H 1800 2750 50  0001 C CNN
@@
 $EndComp
 $Comp
-L CUSTOM_COMPONENTS:R_C R51
+L VIOBOARD-rescue:R_C-CUSTOM_COMPONENTS R51
 U 1 1 599865B4
 P 1800 2850
 F 0 "R51" V 1800 2850 39  0000 C CNN
-F 1 "470 1%" V 1750 2600 39  0000 C CNN
+F 1 "470" V 1750 2600 39  0000 C CNN
 F 2 "Resistors_SMD:R_0805" V 1730 2850 50  0001 C CNN
 F 3 "" H 1800 2850 50  0001 C CNN
@@
 $EndComp
 $Comp
-L CUSTOM_COMPONENTS:R_C R52
+L VIOBOARD-rescue:R_C-CUSTOM_COMPONENTS R52
 U 1 1 599865FD
 P 1800 2950
 F 0 "R52" V 1800 2950 39  0000 C CNN
-F 1 "470 1%" V 1750 2700 39  0000 C CNN
+F 1 "470" V 1750 2700 39  0000 C CNN
 F 2 "Resistors_SMD:R_0805" V 1730 2950 50  0001 C CNN
 F 3 "" H 1800 2950 50  0001 C CNN
@@
 P 8650 4550
 F 0 "R61" V 8650 4550 50  0000 C CNN
-F 1 "100 1%" V 8550 4550 39  0000 C CNN
+F 1 "100" V 8550 4550 39  0000 C CNN
 F 2 "Resistors_SMD:R_0805" V 8580 4550 50  0001 C CNN
 F 3 "" H 8650 4550 50  0001 C CNN
@@
 P 8650 4750
 F 0 "R62" V 8650 4750 50  0000 C CNN
-F 1 "100 1%" V 8550 4750 39  0000 C CNN
+F 1 "100" V 8550 4750 39  0000 C CNN
 F 2 "Resistors_SMD:R_0805" V 8580 4750 50  0001 C CNN
 F 3 "" H 8650 4750 50  0001 C CNN
@@
 P 8650 4950
 F 0 "R63" V 8650 4950 50  0000 C CNN
-F 1 "100 1%" V 8550 4950 39  0000 C CNN
+F 1 "100" V 8550 4950 39  0000 C CNN
 F 2 "Resistors_SMD:R_0805" V 8580 4950 50  0001 C CNN
 F 3 "" H 8650 4950 50  0001 C CNN
@@
 P 8650 5150
 F 0 "R64" V 8650 5150 50  0000 C CNN
-F 1 "100 1%" V 8550 5150 39  0000 C CNN
+F 1 "100" V 8550 5150 39  0000 C CNN
 F 2 "Resistors_SMD:R_0805" V 8580 5150 50  0001 C CNN
 F 3 "" H 8650 5150 50  0001 C CNN
@@
 P 6350 5800
 F 0 "R86" H 6380 5820 50  0000 L CNN
-F 1 "4.7K 1%" H 6050 5800 39  0000 L CNN
+F 1 "4K7" H 6050 5800 39  0000 L CNN
 F 2 "Resistors_SMD:R_0805" H 6350 5800 50  0001 C CNN
 F 3 "" H 6350 5800 50  0001 C CNN
@@
 P 6450 6000
 F 0 "R87" H 6480 6020 50  0000 L CNN
-F 1 "4.7K 1%" H 6050 6000 39  0000 L CNN
+F 1 "4K7" H 6050 6000 39  0000 L CNN
 F 2 "Resistors_SMD:R_0805" H 6450 6000 50  0001 C CNN
 F 3 "" H 6450 6000 50  0001 C CNN
@@
 P 6550 6200
 F 0 "R88" H 6580 6220 50  0000 L CNN
-F 1 "4.7K 1%" H 6050 6200 39  0000 L CNN
+F 1 "4K7" H 6050 6200 39  0000 L CNN
 F 2 "Resistors_SMD:R_0805" H 6550 6200 50  0001 C CNN
 F 3 "" H 6550 6200 50  0001 C CNN
@@
 P 6650 6400
 F 0 "R89" H 6680 6420 50  0000 L CNN
-F 1 "4.7K 1%" H 6050 6400 39  0000 L CNN
+F 1 "4K7" H 6050 6400 39  0000 L CNN
 F 2 "Resistors_SMD:R_0805" H 6650 6400 50  0001 C CNN
 F 3 "" H 6650 6400 50  0001 C CNN
