File: VIOBOARD/IOCONTROLLER.sch (KiCad schematic (older format))
At the start: 6 parts, among them J20 CONN_01X06, Y2 10MHz

Commit message: Libraries modified as part of the BBB cape developement.
Parts:
- C18, C19: symbol device:C_Small -> VIOBOARD-rescue:C_Small-device
- Y2: symbol device:Crystal -> VIOBOARD-rescue:Crystal-device
Changed lines of the file:
@@
 $EndDescr
 $Comp
-L device:C_Small C18
+L VIOBOARD-rescue:C_Small-device C18
 U 1 1 59155B56
 P 6700 3300
@@
 $EndComp
 $Comp
-L device:C_Small C19
+L VIOBOARD-rescue:C_Small-device C19
 U 1 1 59155B5D
 P 6700 3600
@@
 $EndComp
 $Comp
-L device:Crystal Y2
+L VIOBOARD-rescue:Crystal-device Y2
 U 1 1 59155B64
 P 6400 3450

Commit message: Schematics cleanup.  Gerbers for the latest manufacturing release.
Parts:
- R10: value 10K 1% -> 10K; symbol CUSTOM_COMPONENTS:R_C -> VIOBOARD-rescue:R_C-CUSTOM_COMPONENTS
- dsPIC1: symbol CUSTOM_COMPONENTS:dsPIC30F4013 -> VIOBOARD-rescue:dsPIC30F4013-CUSTOM_COMPONENTS
Changed lines of the file:
@@
 $EndComp
 $Comp
-L CUSTOM_COMPONENTS:R_C R10
+L VIOBOARD-rescue:R_C-CUSTOM_COMPONENTS R10
 U 1 1 59155BBE
 P 5600 4850
 F 0 "R10" V 5600 4850 50  0000 C CNN
-F 1 "10K 1%" V 5500 4850 39  0000 C CNN
+F 1 "10K" V 5500 4850 39  0000 C CNN
 F 2 "Resistors_SMD:R_0805" V 5530 4850 50  0001 C CNN
 F 3 "" H 5600 4850 50  0001 C CNN
@@
 RB9/AN9/ICD1
 $Comp
-L CUSTOM_COMPONENTS:dsPIC30F4013 dsPIC1
+L VIOBOARD-rescue:dsPIC30F4013-CUSTOM_COMPONENTS dsPIC1
 U 1 1 59155B6B
 P 4350 4500
