File: VIOBOARD/MAX232.sch (KiCad schematic (older format))
At the start: 6 parts, among them U1 MAX232I

Commit message: Libraries modified as part of the BBB cape developement.
Parts:
- C60, C61, C62, C63, C64: symbol device:C_Small -> VIOBOARD-rescue:C_Small-device
- U1: symbol interface:MAX232I -> VIOBOARD-rescue:MAX232I-interface
Changed lines of the file:
@@
 $EndDescr
 $Comp
-L interface:MAX232I U1
+L VIOBOARD-rescue:MAX232I-interface U1
 U 1 1 5A48FCB4
 P 5650 3700
@@
 $EndComp
 $Comp
-L device:C_Small C60
+L VIOBOARD-rescue:C_Small-device C60
 U 1 1 5A48FE6E
 P 4550 2950
@@
 $EndComp
 $Comp
-L device:C_Small C61
+L VIOBOARD-rescue:C_Small-device C61
 U 1 1 5A48FEAC
 P 6600 2950
@@
 $EndComp
 $Comp
-L device:C_Small C62
+L VIOBOARD-rescue:C_Small-device C62
 U 1 1 5A490198
 P 6750 3300
@@
 $EndComp
 $Comp
-L device:C_Small C63
+L VIOBOARD-rescue:C_Small-device C63
 U 1 1 5A4901D4
 P 6750 3600
@@
 	4550 3100 4850 3100
 $Comp
-L device:C_Small C64
+L VIOBOARD-rescue:C_Small-device C64
 U 1 1 5A490CAE
 P 7500 2550

Commit message: Schematics cleanup.  Gerbers for the latest manufacturing release.
Changed lines of the file:
@@
 	6850 3600 7050 3600
 Wire Wire Line
-	7050 3600 7050 3300
+	7050 3600 7050 3450
 Wire Wire Line
 	7050 3300 6850 3300
@@
 	5650 2500 5650 2350
 Wire Wire Line
-	5400 2350 7500 2350
+	5400 2350 5650 2350
 Wire Wire Line
 	7500 2350 7500 2450
@@
 Wire Wire Line
 	7350 4400 6450 4400
+Wire Wire Line
+	7050 3450 7050 3300
+Wire Wire Line
+	5650 2350 7500 2350
 $EndSCHEMATC
