File: VIOBOARD/MIC5013.sch (KiCad schematic (older format))
At the start: 14 parts, among them Q1 RFD3055LE, U2 MIC5013

Commit message: Libraries modified as part of the BBB cape developement.
Parts:
- C20: symbol device:C_Small -> VIOBOARD-rescue:C_Small-device
- LED1, LED12: symbol device:LED_ALT -> VIOBOARD-rescue:LED_ALT-device
- Q1: symbol device:Q_NMOS_GDS -> VIOBOARD-rescue:Q_NMOS_GDS-device
Changed lines of the file:
@@
 $EndComp
 $Comp
-L device:Q_NMOS_GDS Q1
+L VIOBOARD-rescue:Q_NMOS_GDS-device Q1
 U 1 1 59672963
 P 6450 3150
@@
 	6550 3350 6550 3600
 $Comp
-L device:C_Small C20
+L VIOBOARD-rescue:C_Small-device C20
 U 1 1 59672976
 P 7500 3050
@@
 	4800 3350 4800 3250
 $Comp
-L device:LED_ALT LED12
+L VIOBOARD-rescue:LED_ALT-device LED12
 U 1 1 596729BF
 P 6550 5350
@@
 $EndComp
 $Comp
-L device:LED_ALT LED1
+L VIOBOARD-rescue:LED_ALT-device LED1
 U 1 1 596958E9
 P 4950 1750

Commit message: Schematics cleanup.  Gerbers for the latest manufacturing release.
Parts:
- R11, R12: value 10K 1% -> 10K; symbol CUSTOM_COMPONENTS:R_C -> VIOBOARD-rescue:R_C-CUSTOM_COMPONENTS
- R13: value 8.2K 1% -> 8K2; symbol CUSTOM_COMPONENTS:R_C -> VIOBOARD-rescue:R_C-CUSTOM_COMPONENTS
- R14: value 2.2K 1% -> 2K2; symbol CUSTOM_COMPONENTS:R_C -> VIOBOARD-rescue:R_C-CUSTOM_COMPONENTS
- R15: value 470 1% -> 470; symbol CUSTOM_COMPONENTS:R_C -> VIOBOARD-rescue:R_C-CUSTOM_COMPONENTS
- R16: value 24K 1% -> 24K; symbol CUSTOM_COMPONENTS:R_C -> VIOBOARD-rescue:R_C-CUSTOM_COMPONENTS
- R17: value 100 1% -> 100; symbol CUSTOM_COMPONENTS:R_C -> VIOBOARD-rescue:R_C-CUSTOM_COMPONENTS
- R18: value 3 1% -> 3; symbol CUSTOM_COMPONENTS:R_C -> VIOBOARD-rescue:R_C-CUSTOM_COMPONENTS
- R19: value 4.7K 1% -> 4K7; symbol CUSTOM_COMPONENTS:R_C -> VIOBOARD-rescue:R_C-CUSTOM_COMPONENTS
- U2: symbol CUSTOM_COMPONENTS:MIC5013 -> VIOBOARD-rescue:MIC5013-CUSTOM_COMPONENTS
Changed lines of the file:
@@
 VDD_24V_PROT
 $Comp
-L CUSTOM_COMPONENTS:MIC5013 U2
+L VIOBOARD-rescue:MIC5013-CUSTOM_COMPONENTS U2
 U 1 1 5967295C
 P 4050 3250
@@
 	4800 3150 6250 3150
 $Comp
-L CUSTOM_COMPONENTS:R_C R18
+L VIOBOARD-rescue:R_C-CUSTOM_COMPONENTS R18
 U 1 1 5967296D
 P 6550 3750
@@
 AR Path="/59154FA7/592EA18F/5968C780/5967296D" Ref="R43"  Part="1"
 F 0 "R18" V 6550 3750 50  0000 C CNN
-F 1 "3 1%" V 6450 3750 39  0000 C CNN
+F 1 "3" V 6450 3750 39  0000 C CNN
 F 2 "Resistors_SMD:R_0805" V 6480 3750 50  0001 C CNN
 F 3 "" H 6550 3750 50  0001 C CNN
@@
 AR Path="/59154FA7/59251B3A/59266621/5967059A/5967297E" Ref="#PWR018"  Part="1"
 AR Path="/59154FA7/592EA18F/5968C780/5967297E" Ref="#PWR036"  Part="1"
-F 0 "#PWR036" H 7500 3000 50  0001 C CNN
+F 0 "#PWR018" H 7500 3000 50  0001 C CNN
 F 1 "GND" H 7500 3100 50  0000 C CNN
 F 2 "" H 7500 3250 50  0001 C CNN
@@
 Connection ~ 6550 4900
 $Comp
-L CUSTOM_COMPONENTS:R_C R17
+L VIOBOARD-rescue:R_C-CUSTOM_COMPONENTS R17
 U 1 1 5967298E
 P 6000 3550
@@
 AR Path="/59154FA7/592EA18F/5968C780/5967298E" Ref="R42"  Part="1"
 F 0 "R17" V 6000 3550 50  0000 C CNN
-F 1 "100 1%" V 5900 3550 39  0000 C CNN
+F 1 "100" V 5900 3550 39  0000 C CNN
 F 2 "Resistors_SMD:R_0805" V 5930 3550 50  0001 C CNN
 F 3 "" H 6000 3550 50  0001 C CNN
@@
 $EndComp
 $Comp
-L CUSTOM_COMPONENTS:R_C R16
+L VIOBOARD-rescue:R_C-CUSTOM_COMPONENTS R16
 U 1 1 59672995
 P 5700 3900
@@
 AR Path="/59154FA7/592EA18F/5968C780/59672995" Ref="R41"  Part="1"
 F 0 "R16" V 5700 3900 50  0000 C CNN
-F 1 "24K 1%" V 5600 3900 39  0000 C CNN
+F 1 "24K" V 5600 3900 39  0000 C CNN
 F 2 "Resistors_SMD:R_0805" V 5630 3900 50  0001 C CNN
 F 3 "" H 5700 3900 50  0001 C CNN
@@
 AR Path="/59154FA7/59251B3A/59266621/5967059A/596729A2" Ref="#PWR019"  Part="1"
 AR Path="/59154FA7/592EA18F/5968C780/596729A2" Ref="#PWR037"  Part="1"
-F 0 "#PWR037" H 5700 3900 50  0001 C CNN
+F 0 "#PWR019" H 5700 3900 50  0001 C CNN
 F 1 "GND" H 5700 4000 50  0000 C CNN
 F 2 "" H 5700 4150 50  0001 C CNN
@@
 	3850 3050 3500 3050
 $Comp
-L CUSTOM_COMPONENTS:R_C R12
+L VIOBOARD-rescue:R_C-CUSTOM_COMPONENTS R12
 U 1 1 596729A9
 P 3350 3050
@@
 AR Path="/59154FA7/592EA18F/5968C780/596729A9" Ref="R37"  Part="1"
 F 0 "R12" V 3350 3050 39  0000 C CNN
-F 1 "10K 1%" V 3450 3050 39  0000 C CNN
+F 1 "10K" V 3450 3050 39  0000 C CNN
 F 2 "Resistors_SMD:R_0805" V 3280 3050 50  0001 C CNN
 F 3 "" H 3350 3050 50  0001 C CNN
@@
 AR Path="/59154FA7/59251B3A/59266621/5967059A/596729B2" Ref="#PWR020"  Part="1"
 AR Path="/59154FA7/592EA18F/5968C780/596729B2" Ref="#PWR038"  Part="1"
-F 0 "#PWR038" H 3200 3450 50  0001 C CNN
+F 0 "#PWR020" H 3200 3450 50  0001 C CNN
 F 1 "GND" H 3200 3550 50  0000 C CNN
 F 2 "" H 3200 3700 50  0001 C CNN
@@
 AR Path="/59154FA7/59251B3A/59266621/5967059A/596729B8" Ref="#PWR021"  Part="1"
 AR Path="/59154FA7/592EA18F/5968C780/596729B8" Ref="#PWR039"  Part="1"
-F 0 "#PWR039" H 4800 3100 50  0001 C CNN
+F 0 "#PWR021" H 4800 3100 50  0001 C CNN
 F 1 "GND" H 4800 3200 50  0000 C CNN
 F 2 "" H 4800 3350 50  0001 C CNN
@@
 $EndComp
 $Comp
-L CUSTOM_COMPONENTS:R_C R19
+L VIOBOARD-rescue:R_C-CUSTOM_COMPONENTS R19
 U 1 1 596729C6
 P 6550 5800
@@
 AR Path="/59154FA7/592EA18F/5968C780/596729C6" Ref="R44"  Part="1"
 F 0 "R19" V 6550 5800 39  0000 C CNN
-F 1 "4.7K 1%" V 6450 5800 39  0000 C CNN
+F 1 "4K7" V 6450 5800 39  0000 C CNN
 F 2 "Resistors_SMD:R_0805" V 6480 5800 50  0001 C CNN
 F 3 "" H 6550 5800 50  0001 C CNN
@@
 AR Path="/59154FA7/59251B3A/59266621/5967059A/596729CD" Ref="#PWR022"  Part="1"
 AR Path="/59154FA7/592EA18F/5968C780/596729CD" Ref="#PWR040"  Part="1"
-F 0 "#PWR040" H 6550 5850 50  0001 C CNN
+F 0 "#PWR022" H 6550 5850 50  0001 C CNN
 F 1 "GND" H 6550 5950 50  0000 C CNN
 F 2 "" H 6550 6100 50  0001 C CNN
@@
 AR Path="/59154FA7/59251B3A/59266621/5967059A/5968D26F" Ref="#FLG023"  Part="1"
 AR Path="/59154FA7/592EA18F/5968C780/5968D26F" Ref="#FLG041"  Part="1"
-F 0 "#FLG041" H 8400 4800 50  0001 C CNN
+F 0 "#FLG023" H 8400 4800 50  0001 C CNN
 F 1 "PWR_FLAG" H 8400 5050 50  0000 C CNN
 F 2 "" H 8400 4900 50  0001 C CNN
@@
 Connection ~ 8400 4900
 $Comp
-L CUSTOM_COMPONENTS:R_C R13
+L VIOBOARD-rescue:R_C-CUSTOM_COMPONENTS R13
 U 1 1 5969557C
 P 4950 2500
@@
 AR Path="/59154FA7/592EA18F/5968C780/5969557C" Ref="R38"  Part="1"
 F 0 "R13" V 4950 2500 39  0000 C CNN
-F 1 "8.2K 1%" V 5050 2500 39  0000 C CNN
+F 1 "8K2" V 5050 2500 39  0000 C CNN
 F 2 "Resistors_SMD:R_0805" V 4880 2500 50  0001 C CNN
 F 3 "" H 4950 2500 50  0001 C CNN
@@
 $EndComp
 $Comp
-L CUSTOM_COMPONENTS:R_C R14
+L VIOBOARD-rescue:R_C-CUSTOM_COMPONENTS R14
 U 1 1 596955EB
 P 5250 2500
@@
 AR Path="/59154FA7/592EA18F/5968C780/596955EB" Ref="R39"  Part="1"
 F 0 "R14" V 5250 2500 39  0000 C CNN
-F 1 "2.2K 1%" V 5350 2500 39  0000 C CNN
+F 1 "2K2" V 5350 2500 39  0000 C CNN
 F 2 "Resistors_SMD:R_0805" V 5180 2500 50  0001 C CNN
 F 3 "" H 5250 2500 50  0001 C CNN
@@
 AR Path="/59154FA7/59251B3A/59266621/5967059A/5969571B" Ref="#PWR024"  Part="1"
 AR Path="/59154FA7/592EA18F/5968C780/5969571B" Ref="#PWR042"  Part="1"
-F 0 "#PWR042" H 5400 2550 50  0001 C CNN
+F 0 "#PWR024" H 5400 2550 50  0001 C CNN
 F 1 "GND" H 5400 2650 50  0000 C CNN
 F 2 "" H 5400 2800 50  0001 C CNN
@@
 	5400 2200 5400 2800
 $Comp
-L CUSTOM_COMPONENTS:R_C R15
+L VIOBOARD-rescue:R_C-CUSTOM_COMPONENTS R15
 U 1 1 5969589C
 P 5400 2050
@@
 AR Path="/59154FA7/592B5967/5969589C" Ref="R40"  Part="1"
 F 0 "R15" V 5400 2050 50  0000 C CNN
-F 1 "470 1%" V 5300 2050 39  0000 C CNN
+F 1 "470" V 5300 2050 39  0000 C CNN
 F 2 "Resistors_SMD:R_0805" V 5330 2050 50  0001 C CNN
 F 3 "" H 5400 2050 50  0001 C CNN
@@
 	1800 2950 3850 2950
 $Comp
-L CUSTOM_COMPONENTS:R_C R11
+L VIOBOARD-rescue:R_C-CUSTOM_COMPONENTS R11
 U 1 1 596ADB60
 P 2350 3100
@@
 AR Path="/59154FA7/592EA18F/5968C780/596ADB60" Ref="R36"  Part="1"
 F 0 "R11" V 2350 3100 50  0000 C CNN
-F 1 "10K 1%" V 2250 3100 39  0000 C CNN
+F 1 "10K" V 2250 3100 39  0000 C CNN
 F 2 "Resistors_SMD:R_0805" V 2280 3100 50  0001 C CNN
 F 3 "" H 2350 3100 50  0001 C CNN
@@
 AR Path="/59154FA7/592EA18F/5968C780/59965072" Ref="#PWR043"  Part="1"
 AR Path="/59154FA7/59251B3A/59266621/5967059A/59965072" Ref="#PWR025"  Part="1"
-F 0 "#PWR043" H 2350 3150 50  0001 C CNN
+F 0 "#PWR025" H 2350 3150 50  0001 C CNN
 F 1 "GND" H 2350 3250 50  0000 C CNN
 F 2 "" H 2350 3400 50  0001 C CNN
