File: VIOBOARD/STATUS_LEDS.sch (KiCad schematic (older format))
At the start: 8 parts

Commit message: Libraries modified as part of the BBB cape developement.
Parts:
- LED2, LED3, LED4, LED5: symbol device:LED_ALT -> VIOBOARD-rescue:LED_ALT-device
Changed lines of the file:
@@
 $EndDescr
 $Comp
-L device:LED_ALT LED2
+L VIOBOARD-rescue:LED_ALT-device LED2
 U 1 1 592B5DE2
 P 4750 2600
@@
 $EndComp
 $Comp
-L device:LED_ALT LED3
+L VIOBOARD-rescue:LED_ALT-device LED3
 U 1 1 592B5DF0
 P 4750 2900
@@
 $EndComp
 $Comp
-L device:LED_ALT LED4
+L VIOBOARD-rescue:LED_ALT-device LED4
 U 1 1 592B5DF7
 P 4750 3300
@@
 $EndComp
 $Comp
-L device:LED_ALT LED5
+L VIOBOARD-rescue:LED_ALT-device LED5
 U 1 1 592B5DFE
 P 4750 3650

Commit message: Schematics cleanup.  Gerbers for the latest manufacturing release.
Parts:
- R1, R46, R47, R48: value 470 1% -> 470; symbol CUSTOM_COMPONENTS:R_C -> VIOBOARD-rescue:R_C-CUSTOM_COMPONENTS
Changed lines of the file:
@@
 	6300 3300 6300 3450
 $Comp
-L CUSTOM_COMPONENTS:R_C R1
+L VIOBOARD-rescue:R_C-CUSTOM_COMPONENTS R1
 U 1 1 59969F73
 P 5200 2600
 F 0 "R1" V 5200 2600 50  0000 C CNN
-F 1 "470 1%" V 5100 2600 39  0000 C CNN
+F 1 "470" V 5100 2600 39  0000 C CNN
 F 2 "Resistors_SMD:R_0805" V 5130 2600 50  0001 C CNN
 F 3 "" H 5200 2600 50  0001 C CNN
@@
 $EndComp
 $Comp
-L CUSTOM_COMPONENTS:R_C R46
+L VIOBOARD-rescue:R_C-CUSTOM_COMPONENTS R46
 U 1 1 59969FE4
 P 5200 2900
 F 0 "R46" V 5200 2900 50  0000 C CNN
-F 1 "470 1%" V 5100 2900 39  0000 C CNN
+F 1 "470" V 5100 2900 39  0000 C CNN
 F 2 "Resistors_SMD:R_0805" V 5130 2900 50  0001 C CNN
 F 3 "" H 5200 2900 50  0001 C CNN
@@
 $EndComp
 $Comp
-L CUSTOM_COMPONENTS:R_C R47
+L VIOBOARD-rescue:R_C-CUSTOM_COMPONENTS R47
 U 1 1 5996A033
 P 5200 3300
 F 0 "R47" V 5200 3300 50  0000 C CNN
-F 1 "470 1%" V 5100 3300 39  0000 C CNN
+F 1 "470" V 5100 3300 39  0000 C CNN
 F 2 "Resistors_SMD:R_0805" V 5130 3300 50  0001 C CNN
 F 3 "" H 5200 3300 50  0001 C CNN
@@
 $EndComp
 $Comp
-L CUSTOM_COMPONENTS:R_C R48
+L VIOBOARD-rescue:R_C-CUSTOM_COMPONENTS R48
 U 1 1 5996A07A
 P 5200 3650
 F 0 "R48" V 5200 3650 50  0000 C CNN
-F 1 "470 1%" V 5100 3650 39  0000 C CNN
+F 1 "470" V 5100 3650 39  0000 C CNN
 F 2 "Resistors_SMD:R_0805" V 5130 3650 50  0001 C CNN
 F 3 "" H 5200 3650 50  0001 C CNN
