File: VIOBOARD/VREF+.sch (KiCad schematic (older format))
At the start: 4 parts, among them J10 TEST_1P, U7 REF02CSZ

Commit message: Libraries modified as part of the BBB cape developement.
Parts:
- C42, C43: symbol device:C_Small -> VIOBOARD-rescue:C_Small-device
- J10: symbol conn:TEST_1P -> VIOBOARD-rescue:TEST_1P-conn
Changed lines of the file:
@@
 	5150 2800 6150 2800
 $Comp
-L device:C_Small C42
+L VIOBOARD-rescue:C_Small-device C42
 U 1 1 5968DF52
 P 3500 3000
@@
 	3500 3250 3500 3100
 $Comp
-L device:C_Small C43
+L VIOBOARD-rescue:C_Small-device C43
 U 1 1 5968E10A
 P 5700 3000
@@
 	5700 3250 5700 3100
 $Comp
-L conn:TEST_1P J10
+L VIOBOARD-rescue:TEST_1P-conn J10
 U 1 1 596A8A07
 P 5700 2800

Commit message: Schematics cleanup.  Gerbers for the latest manufacturing release.
Parts:
- U7: symbol CUSTOM_COMPONENTS:REF02CSZ -> VIOBOARD-rescue:REF02CSZ-CUSTOM_COMPONENTS
Changed lines of the file:
@@
 $EndDescr
 $Comp
-L CUSTOM_COMPONENTS:REF02CSZ U7
+L VIOBOARD-rescue:REF02CSZ-CUSTOM_COMPONENTS U7
 U 1 1 5968CC43
 P 4550 3050
@@
 VREF+
 Wire Wire Line
-	3000 2700 4350 2700
+	3000 2700 3500 2700
 Wire Wire Line
-	5150 2800 6150 2800
+	5150 2800 5700 2800
 $Comp
 L VIOBOARD-rescue:C_Small-device C42
@@
 	1    0    0    -1
 $EndComp
+Wire Wire Line
+	3500 2700 4350 2700
+Wire Wire Line
+	5700 2800 6150 2800
 $EndSCHEMATC
