File: VIOBOARD/comm_controller.sch (KiCad schematic (older format))
At the start: 19 parts, among them J12 TP SCL, J13 TP SDA, J14 TP_CTS, J15 TP_TD, J16 TP_RTS, J17 TP_RD, J18 TP_GND, J19 CONN_01X06, J3 BOARD_COMM, Y1 8MHz

Commit message: Libraries modified as part of the BBB cape developement.
Parts:
- C6, C7, C8: symbol device:C_Small -> VIOBOARD-rescue:C_Small-device
- J12, J13, J14, J15, J16, J17, J18: symbol conn:TEST_1P -> VIOBOARD-rescue:TEST_1P-conn
- LED14: symbol device:LED_ALT -> VIOBOARD-rescue:LED_ALT-device
- Y1: symbol device:Crystal -> VIOBOARD-rescue:Crystal-device
Connections:
- wire segments 70 -> 84
Changed lines of the file:
@@
 $EndComp
 $Comp
-L device:LED_ALT LED14
+L VIOBOARD-rescue:LED_ALT-device LED14
 U 1 1 5915ADE3
 P 8700 2800
@@
 $EndComp
 $Comp
-L device:Crystal Y1
+L VIOBOARD-rescue:Crystal-device Y1
 U 1 1 5915ADFF
 P 4300 3450
@@
 NoConn ~ 6650 2700
 $Comp
-L device:C_Small C6
+L VIOBOARD-rescue:C_Small-device C6
 U 1 1 5915AE2B
 P 3250 3300
@@
 $EndComp
 $Comp
-L device:C_Small C7
+L VIOBOARD-rescue:C_Small-device C7
 U 1 1 5915AE32
 P 3250 3700
@@
 	4500 3700 4500 3400
 Wire Wire Line
-	3350 3300 5400 3300
+	3350 3300 4300 3300
 Connection ~ 4300 3300
-Connection ~ 4300 3600
 Wire Wire Line
 	5400 3000 4950 3000
@@
 	6650 4350 6650 3800
 Wire Wire Line
-	1600 1050 1600 4350
+	1600 1050 1600 1150
 Wire Wire Line
 	1600 4350 6650 4350
@@
 	5250 4200 2000 4200
 Wire Wire Line
-	2000 4200 2000 1050
-Wire Wire Line
-	3350 3700 4500 3700
+	2000 4200 2000 1450
+Wire Wire Line
+	3350 3700 4300 3700
 Wire Wire Line
 	4300 3600 4300 3700
@@
 	3150 3300 2900 3300
 Wire Wire Line
-	6600 5500 8350 5500
-Wire Wire Line
-	6600 5400 8350 5400
-Wire Wire Line
-	6600 5600 8350 5600
-Wire Wire Line
-	6600 5700 8350 5700
+	6600 5500 7050 5500
+Wire Wire Line
+	6600 5400 6700 5400
+Wire Wire Line
+	6600 5600 7750 5600
+Wire Wire Line
+	6600 5700 8150 5700
 Wire Wire Line
 	6650 3300 9400 3300
@@
 	4950 1900 4950 2900
 Wire Wire Line
-	5350 1500 5350 2500
-Wire Wire Line
-	5300 2500 5400 2500
+	5350 1500 5350 1900
+Wire Wire Line
+	5300 2500 5350 2500
 Connection ~ 5350 2500
 Wire Wire Line
 	4600 3700 5400 3700
 $Comp
-L device:C_Small C8
+L VIOBOARD-rescue:C_Small-device C8
 U 1 1 591D9DD5
 P 9400 3200
@@
 $EndComp
 Wire Wire Line
-	4150 2500 5000 2500
+	4150 2500 4650 2500
 Connection ~ 1600 1150
 Text Notes 6250 650  0    60   ~ 0
@@
 $EndSheet
 Wire Wire Line
-	9150 2800 9900 2800
+	9150 2800 9400 2800
 Wire Wire Line
 	9400 2800 9400 3100
@@
 	7050 2500 6650 2500
 Wire Wire Line
-	2900 3300 2900 3850
+	2900 3300 2900 3700
 Wire Wire Line
 	5400 3200 4650 3200
@@
 	4600 2800 4600 3700
 Wire Wire Line
-	1000 1450 1700 1450
+	1000 1450 1150 1450
 Wire Wire Line
 	1150 1150 1300 1150
@@
 Connection ~ 5350 1900
 $Comp
-L conn:TEST_1P J14
+L VIOBOARD-rescue:TEST_1P-conn J14
 U 1 1 596AAE0A
 P 6700 6100
+AR Path="/596AAE0A" Ref="J14"  Part="1"
+AR Path="/5915A6A3/596AAE0A" Ref="J14"  Part="1"
 F 0 "J14" H 6700 6370 50  0000 C CNN
 F 1 "TP_CTS" H 6700 6300 39  0000 C CNN
@@
 $EndComp
 $Comp
-L conn:TEST_1P J15
+L VIOBOARD-rescue:TEST_1P-conn J15
 U 1 1 596AAEB3
 P 7050 6100
+AR Path="/596AAEB3" Ref="J15"  Part="1"
+AR Path="/5915A6A3/596AAEB3" Ref="J15"  Part="1"
 F 0 "J15" H 7050 6370 50  0000 C CNN
 F 1 "TP_TD" H 7050 6300 39  0000 C CNN
@@
 $EndComp
 $Comp
-L conn:TEST_1P J16
+L VIOBOARD-rescue:TEST_1P-conn J16
 U 1 1 596AAF6A
 P 7750 4950
+AR Path="/596AAF6A" Ref="J16"  Part="1"
+AR Path="/5915A6A3/596AAF6A" Ref="J16"  Part="1"
 F 0 "J16" H 7750 5220 50  0000 C CNN
 F 1 "TP_RTS" H 7750 5150 39  0000 C CNN
@@
 	8300 5100 8350 5100
 $Comp
-L conn:TEST_1P J17
+L VIOBOARD-rescue:TEST_1P-conn J17
 U 1 1 596ABE4D
 P 8150 4950
+AR Path="/596ABE4D" Ref="J17"  Part="1"
+AR Path="/5915A6A3/596ABE4D" Ref="J17"  Part="1"
 F 0 "J17" H 8150 5220 50  0000 C CNN
 F 1 "TP_RD" H 8150 5150 50  0000 C CNN
@@
 Connection ~ 8150 5700
 $Comp
-L conn:TEST_1P J13
+L VIOBOARD-rescue:TEST_1P-conn J13
 U 1 1 596ACFC7
 P 2000 1450
+AR Path="/596ACFC7" Ref="J13"  Part="1"
+AR Path="/5915A6A3/596ACFC7" Ref="J13"  Part="1"
 F 0 "J13" H 2000 1720 50  0000 C CNN
 F 1 "TP SDA" H 2000 1650 39  0000 C CNN
@@
 $EndComp
 $Comp
-L conn:TEST_1P J12
+L VIOBOARD-rescue:TEST_1P-conn J12
 U 1 1 596AD0C7
 P 1600 1150
+AR Path="/596AD0C7" Ref="J12"  Part="1"
+AR Path="/5915A6A3/596AD0C7" Ref="J12"  Part="1"
 F 0 "J12" H 1600 1420 50  0000 C CNN
 F 1 "TP SCL" H 1600 1350 39  0000 C CNN
@@
 $EndComp
 $Comp
-L conn:TEST_1P J18
+L VIOBOARD-rescue:TEST_1P-conn J18
 U 1 1 596B0B98
 P 9050 4850
+AR Path="/596B0B98" Ref="J18"  Part="1"
+AR Path="/5915A6A3/596B0B98" Ref="J18"  Part="1"
 F 0 "J18" H 9050 5120 50  0000 C CNN
 F 1 "TP_GND" H 9050 5050 39  0000 C CNN
@@
 Text HLabel 5550 1900 2    30   BiDi ~ 0
 COMM_RESET
+Wire Wire Line
+	4300 3300 5400 3300
+Wire Wire Line
+	4300 3700 4500 3700
+Wire Wire Line
+	5350 2500 5400 2500
+Wire Wire Line
+	1600 1150 1600 4350
+Wire Wire Line
+	9400 2800 9900 2800
+Wire Wire Line
+	1150 1450 1700 1450
+Wire Wire Line
+	2900 3700 2900 3850
+Wire Wire Line
+	4650 2500 5000 2500
+Wire Wire Line
+	2000 1450 2000 1050
+Wire Wire Line
+	5350 1900 5350 2500
+Wire Wire Line
+	6700 5400 8350 5400
+Wire Wire Line
+	7050 5500 8350 5500
+Wire Wire Line
+	7750 5600 8350 5600
+Wire Wire Line
+	8150 5700 8350 5700
 $EndSCHEMATC

Commit message: Schematics cleanup.  Gerbers for the latest manufacturing release.
Parts:
- PIC1: symbol CUSTOM_COMPONENTS:PIC24FVXXKA302 -> VIOBOARD-rescue:PIC24FVXXKA302-CUSTOM_COMPONENTS
- R6, R7: value 4.7K 1% -> 4K7; symbol CUSTOM_COMPONENTS:R_C -> VIOBOARD-rescue:R_C-CUSTOM_COMPONENTS
- R8: value 10K 1% -> 10K; symbol CUSTOM_COMPONENTS:R_C -> VIOBOARD-rescue:R_C-CUSTOM_COMPONENTS
- R9: value 470 1% -> 470; symbol CUSTOM_COMPONENTS:R_C -> VIOBOARD-rescue:R_C-CUSTOM_COMPONENTS
Changed lines of the file:
@@
 $EndDescr
 $Comp
-L CUSTOM_COMPONENTS:PIC24FVXXKA302 PIC1
+L VIOBOARD-rescue:PIC24FVXXKA302-CUSTOM_COMPONENTS PIC1
 U 1 1 5915ADC0
 P 5150 4650
@@
 RB14 - GPIO
 $Comp
-L CUSTOM_COMPONENTS:R_C R9
+L VIOBOARD-rescue:R_C-CUSTOM_COMPONENTS R9
 U 1 1 5915AE43
 P 9000 2800
 F 0 "R9" V 9000 2800 50  0000 C CNN
-F 1 "470 1%" V 8900 2800 39  0000 C CNN
+F 1 "470" V 8900 2800 39  0000 C CNN
 F 2 "Resistors_SMD:R_0805" V 8930 2800 50  0001 C CNN
 F 3 "" H 9000 2800 50  0001 C CNN
@@
 NoConn ~ 8350 5200
 $Comp
-L CUSTOM_COMPONENTS:R_C R6
+L VIOBOARD-rescue:R_C-CUSTOM_COMPONENTS R6
 U 1 1 59186B3A
 P 1450 1150
 F 0 "R6" V 1530 1150 50  0000 C CNN
-F 1 "4.7K 1%" V 1350 1150 50  0000 C CNN
+F 1 "4K7" V 1350 1150 50  0000 C CNN
 F 2 "Resistors_SMD:R_0805" V 1380 1150 50  0001 C CNN
 F 3 "" H 1450 1150 50  0001 C CNN
@@
 $EndComp
 $Comp
-L CUSTOM_COMPONENTS:R_C R7
+L VIOBOARD-rescue:R_C-CUSTOM_COMPONENTS R7
 U 1 1 59186C1B
 P 1850 1450
 F 0 "R7" V 1930 1450 50  0000 C CNN
-F 1 "4.7K 1%" V 1750 1450 50  0000 C CNN
+F 1 "4K7" V 1750 1450 50  0000 C CNN
 F 2 "Resistors_SMD:R_0805" V 1780 1450 50  0001 C CNN
 F 3 "" H 1850 1450 50  0001 C CNN
@@
 I2C_SDA
 $Comp
-L CUSTOM_COMPONENTS:R_C R8
+L VIOBOARD-rescue:R_C-CUSTOM_COMPONENTS R8
 U 1 1 591A9B98
 P 5150 2500
 F 0 "R8" V 5150 2500 50  0000 C CNN
-F 1 "10K 1%" V 5050 2500 39  0000 C CNN
+F 1 "10K" V 5050 2500 39  0000 C CNN
 F 2 "Resistors_SMD:R_0805" V 5080 2500 50  0001 C CNN
 F 3 "" H 5150 2500 50  0001 C CNN
