File: VIOBOARD/power_protection.sch (KiCad schematic (older format))
At the start: 15 parts

Commit message: Schematics cleanup.  Gerbers for the latest manufacturing release.
Parts:
- R2: value 23.2K 1% -> 49K9; symbol CUSTOM_COMPONENTS:R_C -> VIOBOARD-rescue:R_C-CUSTOM_COMPONENTS
- R3: value 2.49K 1% -> 4K7; symbol CUSTOM_COMPONENTS:R_C -> VIOBOARD-rescue:R_C-CUSTOM_COMPONENTS
- R4: value 910 1% -> 910; symbol CUSTOM_COMPONENTS:R_C -> VIOBOARD-rescue:R_C-CUSTOM_COMPONENTS
- R5: value 4.7K 1% -> 4K7; symbol CUSTOM_COMPONENTS:R_C -> VIOBOARD-rescue:R_C-CUSTOM_COMPONENTS
- R65: value 100 1% -> 100
- TL1: symbol CUSTOM_COMPONENTS:TL431 -> VIOBOARD-rescue:TL431-CUSTOM_COMPONENTS
Other:
- note removed: "Vout = 2.520 @ Vin = 26\nI = 1mA @ 26V"
Changed lines of the file:
@@
 VDD_24V
 $Comp
-L CUSTOM_COMPONENTS:TL431 TL1
+L VIOBOARD-rescue:TL431-CUSTOM_COMPONENTS TL1
 U 1 1 59127DF7
 P 5150 4050
@@
 VDD_24V_PROT
 Wire Wire Line
-	2400 4250 7250 4250
+	2400 4250 2800 4250
 Connection ~ 5500 4250
 Connection ~ 4950 4250
 Connection ~ 6250 4250
 $Comp
-L CUSTOM_COMPONENTS:R_C R4
+L VIOBOARD-rescue:R_C-CUSTOM_COMPONENTS R4
 U 1 1 5912A1D0
 P 5500 3000
 F 0 "R4" V 5500 3000 50  0000 C CNN
-F 1 "910 1%" V 5400 3000 39  0000 C CNN
+F 1 "910" V 5400 3000 39  0000 C CNN
 F 2 "Resistors_SMD:R_0805" V 5430 3000 50  0001 C CNN
 F 3 "" H 5500 3000 50  0001 C CNN
@@
 $EndComp
 $Comp
-L CUSTOM_COMPONENTS:R_C R2
+L VIOBOARD-rescue:R_C-CUSTOM_COMPONENTS R2
 U 1 1 5912A221
 P 4950 3550
 F 0 "R2" V 4950 3550 50  0000 C CNN
-F 1 "23.2K 1%" V 5050 3600 39  0000 C CNN
+F 1 "49K9" V 5050 3600 39  0000 C CNN
 F 2 "Resistors_SMD:R_0805" V 4880 3550 50  0001 C CNN
 F 3 "" H 4950 3550 50  0001 C CNN
@@
 $EndComp
 $Comp
-L CUSTOM_COMPONENTS:R_C R3
+L VIOBOARD-rescue:R_C-CUSTOM_COMPONENTS R3
 U 1 1 5912A25C
 P 4950 3850
 F 0 "R3" V 4950 3850 50  0000 C CNN
-F 1 "2.49K 1%" V 4850 3850 39  0000 C CNN
+F 1 "4K7" V 4850 3850 39  0000 C CNN
 F 2 "Resistors_SMD:R_0805" V 4880 3850 50  0001 C CNN
 F 3 "" H 4950 3850 50  0001 C CNN
@@
 $EndComp
 Wire Wire Line
-	4050 2850 8250 2850
+	4050 2850 4350 2850
 Wire Wire Line
 	4950 3400 4950 2850
 Wire Wire Line
-	4950 3700 5250 3700
-Wire Wire Line
-	2450 2850 3850 2850
+	4950 3700 5200 3700
+Wire Wire Line
+	2450 2850 2800 2850
 Connection ~ 4950 2850
 Connection ~ 5500 2850
@@
 	5500 3150 5500 3350
 $Comp
-L CUSTOM_COMPONENTS:R_C R5
+L VIOBOARD-rescue:R_C-CUSTOM_COMPONENTS R5
 U 1 1 5912AC8B
 P 7250 3750
 F 0 "R5" V 7250 3750 50  0000 C CNN
-F 1 "4.7K 1%" V 7150 3750 39  0000 C CNN
+F 1 "4K7" V 7150 3750 39  0000 C CNN
 F 2 "Resistors_SMD:R_0805" V 7180 3750 50  0001 C CNN
 F 3 "" H 7250 3750 50  0001 C CNN
@@
 	0    1    -1   0
 $EndComp
-Connection ~ 7250 4250
 Connection ~ 7250 2850
 Wire Wire Line
@@
 	1    0    0    -1
 $EndComp
-Text Notes 5250 2550 0    60   ~ 0
-Vout = 2.520 @ Vin = 26\nI = 1mA @ 26V
 Text Notes 7500 3100 3    60   ~ 0
 24V PROT
@@
 P 2800 3000
 F 0 "C1" H 2800 3200 50  0000 L CNN
-F 1 "0.012uF 50V" H 2550 2950 39  0000 L CNN
+F 1 "0.012uF 50V" H 2550 3300 39  0000 L CNN
 F 2 "Capacitors_SMD:C_1206" H 2838 2850 50  0001 C CNN
 F 3 "" H 2800 3000 50  0001 C CNN
@@
 $EndComp
 Wire Wire Line
-	2800 3150 3550 3150
+	2800 3150 3050 3150
 Connection ~ 3050 3150
 Connection ~ 3300 3150
 Wire Wire Line
-	2800 3100 2800 4250
+	2800 3100 2800 3150
 Connection ~ 2800 4250
 Connection ~ 2800 2850
@@
 P 2300 2850
 F 0 "R65" V 2380 2850 50  0000 C CNN
-F 1 "100 1%" V 2200 2850 39  0000 C CNN
+F 1 "100" V 2200 2850 39  0000 C CNN
 F 2 "Resistors_SMD:R_2512" V 2230 2850 50  0001 C CNN
 F 3 "" H 2300 2850 50  0001 C CNN
@@
 	2150 2850 1250 2850
 Connection ~ 4650 2850
+Wire Wire Line
+	5500 4250 6250 4250
+Wire Wire Line
+	4950 4250 5200 4250
+Wire Wire Line
+	6250 4250 7250 4250
+Wire Wire Line
+	4950 2850 5500 2850
+Wire Wire Line
+	5500 2850 6250 2850
+Wire Wire Line
+	6250 2850 7250 2850
+Wire Wire Line
+	7250 2850 8250 2850
+Wire Wire Line
+	5200 4250 5500 4250
+Wire Wire Line
+	5200 3700 5250 3700
+Wire Wire Line
+	3050 3150 3300 3150
+Wire Wire Line
+	3300 3150 3550 3150
+Wire Wire Line
+	2800 4250 4350 4250
+Wire Wire Line
+	2800 2850 3050 2850
+Wire Wire Line
+	3050 2850 3300 2850
+Wire Wire Line
+	3300 2850 3550 2850
+Wire Wire Line
+	3550 2850 3850 2850
+Wire Wire Line
+	4350 2850 4650 2850
+Wire Wire Line
+	4350 4250 4950 4250
+Wire Wire Line
+	2800 3150 2800 4250
+Wire Wire Line
+	4650 2850 4950 2850
 $EndSCHEMATC
