File: BBB_SHIELD_V2/CONTROLLER.sch (KiCad schematic (older format))
At the start: 23 parts, among them J2 Conn_01x06_Male, J3 Conn_01x06_Male, U3 MCP1501_SOT-23-6

Commit message: Changed to high-side switching of power supply to boards.  Changed footprints to SOIC.  Misc other changes.
Parts:
- removed TP10, TP5: TestPoint_2Pole, Connector_PinHeader_1.27mm:PinHeader_1x02_P1.27mm_Vertical, symbol Connector:TestPoint_2Pole
- added TP3V3REF1, TPCLK1: TestPoint, TestPoint:TestPoint_THTPad_D1.0mm_Drill0.5mm, symbol Connector:TestPoint
- C4: renamed from C12; DKPN (none) -> 1276-2928-2-ND; MFG (none) -> SAMSUNG; MFGPN (none) -> CL21B105KBFNFNE; NOTES (none) -> REEL, VER 2018-11-25; TEMPCO (none) -> X7R; VOLTAGE (none) -> 50
- C5: renamed from C14; DKPN (none) -> 1276-2928-2-ND; MFG (none) -> SAMSUNG; MFGPN (none) -> CL21B105KBFNFNE; NOTES (none) -> REEL, VER 2018-11-25; TEMPCO (none) -> X7R; VOLTAGE (none) -> 50
- C6: renamed from C13; value 10uF 10V -> 10uF; DKPN (none) -> 1276-1052-1-ND; MFG (none) -> SAMSUNG; MFGPN (none) -> CL21A106KPFNNNE; NOTES (none) -> CT, VER 2018-12-09; TEMPCO (none) -> X5R; VOLTAGE (none) -> 10
- D4: value LED -> LEDHMI1; MFG (none) -> MISC; NOTES (none) -> CT, VER 2018-11-25; TEMPCO (none) -> NA; VOLTAGE (none) -> NA
- D5: value LED -> LEDHMI2; MFG (none) -> MISC; NOTES (none) -> CT, VER 2018-11-25; TEMPCO (none) -> NA; VOLTAGE (none) -> NA
- D6: value LED -> LEDHMI3; MFG (none) -> MISC; NOTES (none) -> CT, VER 2018-11-25; TEMPCO (none) -> NA; VOLTAGE (none) -> NA
- D7: value LED -> LEDHMI4; MFG (none) -> MISC; NOTES (none) -> CT, VER 2018-11-25; TEMPCO (none) -> NA; VOLTAGE (none) -> NA
- D8: renamed from D3; value LED -> LEDHTBT; MFG (none) -> MISC; NOTES (none) -> CT, VER 2018-11-25; TEMPCO (none) -> NA; VOLTAGE (none) -> NA
- J2, J3: DKPN (none) -> WM4104-ND; MFGPN (none) -> 0022052061; NOTES (none) -> BULK, VER 2018-11-25
- PIC1: footprint Package_SO:TSSOP-28_4.4x9.7mm_P0.65mm -> Package_SO:SOIC-28W_7.5x17.9mm_P1.27mm; DKPN (none) -> PIC24FV32KA302-I/SO-ND; MFG (none) -> MICROCHIP; MFGPN (none) -> PIC24FV32KA302-I/SO
- R10: renamed from R6; value 10K 5% -> 10K; DKPN (none) -> 541-3016-1-ND; MFG (none) -> VISHAY; MFGPN (none) -> CRCW080510K0FKTA; NOTES (none) -> CT, VER 2018-11-25
- R11, R12: value 200 1% -> 200R; DKPN (none) -> 541-4146-1-ND; MFG (none) -> VISHAY; MFGPN (none) -> CRCW0805200RFKEAC; NOTES (none) -> REEL, VER 2018-12-09
- R13: renamed from R7; value 10K 5% -> 10K; DKPN (none) -> 541-3016-1-ND; MFG (none) -> VISHAY; MFGPN (none) -> CRCW080510K0FKTA; NOTES (none) -> CT, VER 2018-11-25
- R14: renamed from R13; value 200 1% -> 200R; DKPN (none) -> 541-4146-1-ND; MFG (none) -> VISHAY; MFGPN (none) -> CRCW0805200RFKEAC; NOTES (none) -> REEL, VER 2018-12-09
- R15: renamed from R14; value 200 1% -> 200R; DKPN (none) -> 541-4146-1-ND; MFG (none) -> VISHAY; MFGPN (none) -> CRCW0805200RFKEAC; NOTES (none) -> REEL, VER 2018-12-09
- R16: renamed from R10; value 200 1% -> 200R; DKPN (none) -> 541-4146-1-ND; MFG (none) -> VISHAY; MFGPN (none) -> CRCW0805200RFKEAC; NOTES (none) -> REEL, VER 2018-12-09
- R17: renamed from R9; value 150 1% -> 200R; DKPN (none) -> 541-4146-1-ND; MFG (none) -> VISHAY; MFGPN (none) -> CRCW0805200RFKEAC; NOTES (none) -> REEL, VER 2018-12-09
- R9: renamed from R8; DKPN (none) -> 541-3016-1-ND; MFG (none) -> VISHAY; MFGPN (none) -> CRCW080510K0FKTA; NOTES (none) -> CT, VER 2018-11-25
- VREF3V1: renamed from U3; DKPN (none) -> MCP1501T-33E/CHYCT-ND; MFGPN (none) -> MCP1501T-33E/CHY; NOTES (none) -> BULK, VER 2018-11-25
Connections:
- net 3V3_REF: now also TP3V3REF1.1
- net at PIC1.10 (RA3): now also TPCLK1.1

Commit message: Schematic cleanup and refinement.
Parts:
- J2, J3: footprint Connector_PinHeader_2.54mm:PinHeader_1x06_P2.54mm_Horizontal -> CUSTOM_FOOTPRINTS:PinHeader_1x06_P2.54mm_Horizontal
Connections:
- net HMI3\RB12: now reaches D7.2 (A), PIC1.23 (RB12)
Changed lines of the file:
@@
 F 0 "J2" V 4710 863 50  0000 R CNN
 F 1 "Conn_01x06_Male" V 4801 863 50  0000 R CNN
-F 2 "Connector_PinHeader_2.54mm:PinHeader_1x06_P2.54mm_Horizontal" H 4650 1250 50  0001 C CNN
+F 2 "CUSTOM_FOOTPRINTS:PinHeader_1x06_P2.54mm_Horizontal" H 4650 1250 50  0001 C CNN
 F 3 "" H 4650 1250 50  0001 C CNN
 F 4 "BULK, VER 2018-11-25" H 0   0   50  0001 C CNN "NOTES"
@@
 F 0 "J3" V 6250 5250 50  0000 R CNN
 F 1 "Conn_01x06_Male" V 6350 5500 50  0000 R CNN
-F 2 "Connector_PinHeader_2.54mm:PinHeader_1x06_P2.54mm_Horizontal" H 6450 5250 50  0001 C CNN
+F 2 "CUSTOM_FOOTPRINTS:PinHeader_1x06_P2.54mm_Horizontal" H 6450 5250 50  0001 C CNN
 F 3 "" H 6450 5250 50  0001 C CNN
 F 4 "BULK, VER 2018-11-25" H 0   0   50  0001 C CNN "NOTES"
@@
 Wire Wire Line
 	5400 3600 5400 3850
+Text Label 7350 3400 0    50   ~ 0
+HMI3\RB12
 $EndSCHEMATC

Commit message: Rev 2 problem fixes.
Parts:
- added R22, R25: 0, Resistor_SMD:R_0805_2012Metric, symbol Device:R_Small
- C4, C5: NOTES REEL, VER 2018-11-25 -> VER,2019-07-17,REEL
- C6: NOTES CT, VER 2018-12-09 -> VER,2019-07-17,CT
- D4: value LEDHMI1 -> LED; NOTES CT, VER 2018-11-25 -> VER,2019-07-16,CT
- D5: value LEDHMI2 -> LED; NOTES CT, VER 2018-11-25 -> VER,2019-07-16,CT
- D6: value LEDHMI3 -> LED; NOTES CT, VER 2018-11-25 -> VER,2019-07-16,CT
- D7: value LEDHMI4 -> LED; NOTES CT, VER 2018-11-25 -> VER,2019-07-16,CT
- D8: value LEDHTBT -> LED; NOTES CT, VER 2018-11-25 -> VER,2019-07-16,CT
- J2, J3: NOTES BULK, VER 2018-11-25 -> VER,2019-07-16,REUSE
- PIC1: NOTES (none) -> VER,2019-07-16,CT
- R10, R13, R9: NOTES CT, VER 2018-11-25 -> VER,2019-07-17,CT
- R11, R12, R14, R15, R16, R17: NOTES REEL, VER 2018-12-09 -> VER,2019-07-17,REEL
- VREF3V1: NOTES BULK, VER 2018-11-25 -> VER,2019-07-16,CT
Connections:
- net GND: now also PIC1.15 (RB6)
- net SCL1: now also PIC1.17 (RB8); no longer PIC1.18 (RB9)
- net SDA1: now also PIC1.18 (RB9); no longer PIC1.19 (RA7)
- net at PIC1.11 (RB4): now also R25.1
- new net: PIC1.19 (RA7), R22.2
- new net _PWR_BUTT: R22.1
- new net _SYS_RESETn: R25.2
- no-connect marks 6 -> 3
Other:
- moved on the sheet: C4, C5, C6, D4, D5, D6, D7, D8, J2, J3, PIC1, R10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

Commit message: Schematics cleanup.  Gerbers for the latest manufacturing release.
Parts:
- R22, R25: value 0 -> 200R; DKPN (none) -> 541-4146-1-ND; MFG (none) -> VISHAY; MFGPN (none) -> CRCW0805200RFKEAC
Changed lines of the file:
@@
 encoding utf-8
 Sheet 4 12
-Title ""
-Date ""
-Rev ""
-Comp ""
-Comment1 ""
+Title "VPSB"
+Date "2019-09-03"
+Rev "V3.0"
+Comp "Vidas Simkus"
+Comment1 "Copyright (C) 2019 Vidas Simkus"
 Comment2 ""
 Comment3 ""
@@
 P 3900 3600
 F 0 "R25" V 3704 3600 50  0000 C CNN
-F 1 "0" V 3795 3600 50  0000 C CNN
+F 1 "200R" V 3795 3600 50  0000 C CNN
 F 2 "Resistor_SMD:R_0805_2012Metric" H 3900 3600 50  0001 C CNN
-F 3 "~" H 3900 3600 50  0001 C CNN
+F 3 "" H 3900 3600 50  0001 C CNN
+F 4 "541-4146-1-ND" H 0   0   50  0001 C CNN "DKPN"
+F 5 "VISHAY" H 0   0   50  0001 C CNN "MFG"
+F 6 "CRCW0805200RFKEAC" H 0   0   50  0001 C CNN "MFGPN"
 	1    3900 3600
 	0    1    1    0
@@
 P 6600 3500
 F 0 "R22" V 6800 3500 50  0000 C CNN
-F 1 "0" V 6700 3500 50  0000 C CNN
+F 1 "200R" V 6700 3500 50  0000 C CNN
 F 2 "Resistor_SMD:R_0805_2012Metric" H 6600 3500 50  0001 C CNN
-F 3 "~" H 6600 3500 50  0001 C CNN
+F 3 "" H 6600 3500 50  0001 C CNN
+F 4 "541-4146-1-ND" H 0   0   50  0001 C CNN "DKPN"
+F 5 "VISHAY" H 0   0   50  0001 C CNN "MFG"
+F 6 "CRCW0805200RFKEAC" H 0   0   50  0001 C CNN "MFGPN"
 	1    6600 3500
 	0    1    1    0
